File: blystl15_board.kicad_pcb (KiCad board)
At the start: 2 copper layers, 45 x 45 mm, 47 parts, among them J1 SSD1306, J2 Conn_02x03_Odd_Even, J5 Conn_01x03, J6 DOCK_PADS, M1 BLYST NANO/L15, SW2 SW_Push, SW3 SW_Push, SW4 SW_Push, U2 MAX30102EFD+T, U3 W25Q80EWSNIG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

Commit message: DRC Errors Cleared
Parts:
- moved R9 0.50 mm to (117.0, 90.5)
Routing:
- net VDD: track 218.4 -> 243.0 mm, vias 13 -> 15
- net GND: track 73.0 -> 86.2 mm, vias 41 -> 42
- net /P1.07  AIN3: track 54.6 -> 55.4 mm
- net /nRESET: track 32.2 -> 32.8 mm
- net /P2.02: track 86.0 -> 86.5 mm, vias 7 -> 6
- net /P0.03: track 63.2 -> 63.3 mm, vias 4 -> 6
- net /Sensors/QVAR_SWIPE: vias 1 -> 0
- net (no net): vias 1 -> 0
Other:
- outline, holes or cut-outs redrawn
